Commit message: Updated gazebo models etc with Kamil's most recent changes. Wrote script to auto-install ORB_SLAM3 dependencies. Added in ORB_SLAM2 ros wrapper, and patched it to use latest ubuntu, open cv, etc. ROS wrapper still not compiling completely. Further changes will be made.

File: catkin_ws/src/jet_description/urdf/jet.xacro (robot description, xacro)
@@ -139,5 +139,5 @@
       <origin xyz="0 0 0" rpy="1.570796327 0 1.570796327"/>
       <mass value="0.1" />
-      <inertia ixx="1e-6" ixy="0" ixz="0" iyy="1e-6" iyz="0" izz="1e-6" />
+      <inertia ixx="0" ixy="0" ixz="0" iyy="0" iyz="0" izz="0" />
     </inertial>
   </link>
@@ -250,5 +250,5 @@
     <axis xyz="1 0 0" rpy="0 0 0"/>
     <limit effort="100" velocity="100"/>
-    <joint_properties damping="1.0" friction="1.0"/>
+    <joint_properties damping="3.0" friction="0.0"/>
   </joint>
   <!-- Right Wheel Joint -->
@@ -259,5 +259,5 @@
     <axis xyz="1 0 0" rpy="0 0 0"/>
     <limit effort="100" velocity="100"/>
-    <joint_properties damping="1.0" friction="1.0"/>
+    <joint_properties damping="3.0" friction="0.0"/>
   </joint>
   <!-- Caster Link Joint -->

Commit message: Updated jet_navigation

File: catkin_ws/src/jet_description/urdf/jet.xacro (robot description, xacro)
@@ -81,5 +81,5 @@
       <origin xyz="0 0 0" rpy="0 0 0"/>
       <geometry>
-        <mesh filename="package://jet_description/meshes/Right_Wheel.dae"/>
+        <mesh filename="package://jet_description/meshes/Left_Wheel.dae"/>
       </geometry>
     </collision>
@@ -250,5 +250,5 @@
     <axis xyz="1 0 0" rpy="0 0 0"/>
     <limit effort="100" velocity="100"/>
-    <joint_properties damping="3.0" friction="0.0"/>
+    <joint_properties damping="1.0" friction="1.0"/>
   </joint>
   <!-- Right Wheel Joint -->
@@ -259,5 +259,5 @@
     <axis xyz="1 0 0" rpy="0 0 0"/>
     <limit effort="100" velocity="100"/>
-    <joint_properties damping="3.0" friction="0.0"/>
+    <joint_properties damping="1.0" friction="1.0"/>
   </joint>
   <!-- Caster Link Joint -->
