Commit message: minor changes in navigation and multi-robot folders, Multi-Robot Exploration working

File: catkin_ws/src/jet_description/urdf/multi_robot.xacro (robot description, xacro)
@@ -9,5 +9,5 @@
      <parent link="Main_Frame"/>
      <child link="chassis"/>
-     <origin xyz="0 0 0" rpy="0 0 0"/>
+     <origin xyz="0 0 0" rpy="0 0 1.570796327"/>
    </joint>
   <!--.........................Chassis...............................-->
@@ -144,5 +144,5 @@
     <axis xyz="1 0 0" rpy="0 0 0"/>
   </joint>
-  <!--................................Camera..................................-->
+  <!--................................Camera..................................
   <link name="camera">
     <inertial>
@@ -157,5 +157,5 @@
     <parent link="chassis"/>
     <child link="camera"/>
-  </joint>
+  </joint>-->
   <!--............................Liadar................................-->
   <link name="hokuyo">
@@ -172,5 +172,5 @@
     <child link="hokuyo"/>
   </joint>
-  <!--............................IMU................................-->
+  <!--............................IMU................................
   <link name="IMU_link">
     <inertial>
@@ -185,4 +185,4 @@
     <parent link="chassis"/>
     <child link="IMU_link"/>
-  </joint>
+  </joint>-->
 </robot>
