Commit message: updated the jet_* and multi_robot folders to include the latest versions from the Gazebo-Robots branch

File: src/jet_description/urdf/jet.xacro (robot description, xacro)
@@ -1,37 +1,98 @@
 <?xml version="1.0"?>
 <robot name="Jet" xmlns:xacro="http://www.ros.org/wiki/xacro">
-  <!-- Import all Gazebo-customization elements, including Gazebo colors -->
   <xacro:include filename="$(find jet_description)/urdf/jet.gazebo"/>
-  <!-- Import Rviz colors -->
-  <xacro:include filename="$(find jet_description)/urdf/materials.xacro"/>
-<!--........................LINKS........................-->
-  <!-- Chassis -->
+  <!--........................Dummy Link.............................-->
+  <link name="Main_Frame">
+   </link>
+   <joint name="Main_Frame_Joint" type="fixed">
+     <parent link="Main_Frame"/>
+     <child link="chassis"/>
+     <origin xyz="0 0 0" rpy="0 0 1.570796327"/>
+   </joint>
+  <!--.........................Chassis...............................-->
   <link name='chassis'>
-    <pose>0 0 0 0 0 0</pose>
+    <collision name='collision'>
+      <origin xyz="0 0 0" rpy="0 0 0"/>
+      <geometry>
+        <mesh filename="package://jet_description/meshes/Chassis.dae"/>
+      </geometry>
+    </collision>
+    <visual name='chassis_visual'>
+      <origin xyz="0 0 0" rpy="0 0 0"/>
+      <geometry>
+        <mesh filename="package://jet_description/meshes/Chassis.dae"/>
+      </geometry>
+    </visual>
     <inertial>
       <mass value="2.5"/>
       <origin xyz="0 0 0" rpy=" 0 0 0"/>
       <inertia
-          ixx="8.85e-3" ixy="0" ixz="0"
-          iyy="27.08e-3" iyz="0"
+          ixx="27.08e-3" ixy="0" ixz="0"
+          iyy="8.85e-3" iyz="0"
           izz="19.27e-3"/>
     </inertial>
-    <collision name='collision'>
-      <origin xyz="0 0 0" rpy="0 0 3.141592654"/>
-      <geometry>
-        <mesh filename="package://jet_description/meshes/Chassis.dae"/>
-      </geometry>
-    </collision>
-    <visual name='chassis_visual'>
-      <origin xyz="0 0 0" rpy="0 0 3.141592654"/>
-      <geometry>
-        <mesh filename="package://jet_description/meshes/Chassis.dae"/>
-      </geometry>
-    </visual>
-  </link>
-  <!-- Caster Link -->
+  </link>
+  <!--..............................Left Wheel..................................-->
+  <link name="left_wheel">
+    <collision name="collision">
+      <origin xyz="0 0 0" rpy="0 1.570796327 0"/>
+      <geometry>
+        <cylinder radius="0.075" length="0.03"/>
+      </geometry>
+    </collision>
+    <visual name="left_wheel_visual">
+      <origin xyz="0 0 0" rpy="0 0 0"/>
+      <geometry>
+        <mesh filename="package://jet_description/meshes/Left_Wheel.dae"/>
+      </geometry>
+    </visual>
+    <inertial>
+      <origin xyz="0 0 0" rpy="0 0 0"/>
+      <mass value="0.75"/>
+      <inertia
+        ixx="3.51e-4" ixy="0.0" ixz="0.0"
+        iyy="1.11e-3" iyz="0.0"
+        izz="1.11e-3"/>
+    </inertial>
+  </link>
+  <joint type="continuous" name="left_wheel_joint">
+    <origin xyz="0.15 -0.1 0.02" rpy="0 0 0"/>
+    <child link="left_wheel"/>
+    <parent link="chassis"/>
+    <axis xyz="1 0 0" rpy="0 0 0"/>
+  </joint>
+  <!--..............................Right Wheel..................................-->
+  <link name="right_wheel">
+    <collision name="collision">
+      <origin xyz="0 0 0" rpy="0 1.570796327 0"/>
+      <geometry>
+        <cylinder radius="0.075" length="0.03"/>
+      </geometry>
+    </collision>
+    <visual name="right_wheel_visual">
+      <origin xyz="0 0 0" rpy="0 0 0"/>
+      <geometry>
+        <mesh filename="package://jet_description/meshes/Right_Wheel.dae"/>
+      </geometry>
+    </visual>
+    <inertial>
+      <origin xyz="0 0 0" rpy="0 0 0"/>
+      <mass value="0.75"/>
+      <inertia
+        ixx="3.51e-4" ixy="0.0" ixz="0.0"
+        iyy="1.11e-3" iyz="0.0"
+        izz="1.11e-3"/>
+    </inertial>
+  </link>
+  <joint type="continuous" name="right_wheel_joint">
+    <origin xyz="-0.15 -0.1 0.02" rpy="0 0 0"/>
+    <child link="right_wheel"/>
+    <parent link="chassis"/>
+    <axis xyz="1 0 0" rpy="0 0 0"/>
+  </joint>
+  <!--..............................Caster Link...............................-->
   <link name="caster_link">
     <collision name="collision">
-      <origin xyz="0 0 0" rpy="0 0 3.141592654"/>
+      <origin xyz="0 0 0" rpy="0 0 0"/>
       <geometry>
         <mesh filename="package://jet_description/meshes/Caster_Link.dae"/>
@@ -39,5 +100,5 @@
     </collision>
     <visual name="caster_link_visual">
-      <origin xyz="0 0 0" rpy="0 0 3.141592654"/>
+      <origin xyz="0 0 0" rpy="0 0 0"/>
       <geometry>
         <mesh filename="package://jet_description/meshes/Caster_Link.dae"/>
@@ -45,5 +106,5 @@
     </visual>
     <inertial>
-      <origin xyz="0 0 0" rpy="0 0 3.141592654"/>
+      <origin xyz="0 0 0" rpy="0 0 0"/>
       <mass value="0.5"/>
       <inertia
@@ -53,56 +114,16 @@
     </inertial>
   </link>
-  <!-- Left Wheel -->
-  <link name="left_wheel">
-    <collision name="collision">
-      <origin xyz="0 0 0" rpy="0 0 0"/>
-      <geometry>
-        <mesh filename="package://jet_description/meshes/Left_Wheel.dae"/>
-      </geometry>
-    </collision>
-    <visual name="left_wheel_visual">
-      <origin xyz="0 0 0" rpy="0 0 0"/>
-      <geometry>
-        <mesh filename="package://jet_description/meshes/Left_Wheel.dae"/>
-      </geometry>
-    </visual>
-    <inertial>
-      <origin xyz="0 0 0" rpy="0 0 0"/>
-      <mass value="0.75"/>
-      <inertia
-        ixx="3.51e-4" ixy="0.0" ixz="0.0"
-        iyy="1.11e-3" iyz="0.0"
-        izz="1.11e-3"/>
-    </inertial>
-  </link>
-  <!-- Right Wheel -->
-  <link name="right_wheel">
-    <collision name="collision">
-      <origin xyz="0 0 0" rpy="0 0 0"/>
-      <geometry>
-        <mesh filename="package://jet_description/meshes/Right_Wheel.dae"/>
-      </geometry>
-    </collision>
-    <visual name="right_wheel_visual">
-      <origin xyz="0 0 0" rpy="0 0 0"/>
-      <geometry>
-        <mesh filename="package://jet_description/meshes/Right_Wheel.dae"/>
-      </geometry>
-    </visual>
-    <inertial>
-      <origin xyz="0 0 0" rpy="0 0 0"/>
-      <mass value="0.75"/>
-      <inertia
-        ixx="3.51e-4" ixy="0.0" ixz="0.0"
-        iyy="1.11e-3" iyz="0.0"
-        izz="1.11e-3"/>
-    </inertial>
-  </link>
-  <!-- Caster Wheel -->
+  <joint type="continuous" name="caster_joint">
+    <origin xyz="0 0.1 0.005" rpy="0 0 0"/>
+    <child link="caster_link"/>
+    <parent link="chassis"/>
+    <axis xyz="0 0 1" rpy="0 0 0"/>
+  </joint>
+  <!--..............................Caster Wheel..................................-->
   <link name="caster_wheel">
     <collision name="collision">
-      <origin xyz="0 0 0" rpy="0 0 0"/>
-      <geometry>
-        <mesh filename="package://jet_description/meshes/Caster_Wheel.dae"/>
+      <origin xyz="0 0 0" rpy="0 1.570796327 0"/>
+      <geometry>
+        <cylinder radius="0.0225" length="0.015"/>
       </geometry>
     </collision>
@@ -122,153 +143,4 @@
     </inertial>
   </link>
-  <!-- Camera -->
-  <link name="camera">
-    <collision name="collision">
-      <origin xyz="0 0 0" rpy="1.570796327 0 1.570796327"/>
-      <geometry>
-        <mesh filename="package://jet_description/meshes/Camera.dae"/>
-      </geometry>
-    </collision>
-    <visual name="camera_visual">
-      <origin xyz="0 0 0" rpy="1.570796327 0 1.570796327"/>
-      <geometry>
-        <mesh filename="package://jet_description/meshes/Camera.dae"/>
-      </geometry>
-    </visual>
-    <inertial>
-      <origin xyz="0 0 0" rpy="1.570796327 0 1.570796327"/>
-      <mass value="0.1" />
-      <inertia ixx="0" ixy="0" ixz="0" iyy="0" iyz="0" izz="0" />
-    </inertial>
-  </link>
-  <!-- Sonar_Sensor_1 -->
-  <link name="sonar1_link">
-    <collision name="collision">
-      <origin xyz="0 0 0" rpy="0 0 -1.570796327"/>
-      <geometry>
-        <mesh filename="package://jet_description/meshes/Sonar_1.dae"/>
-      </geometry>
-    </collision>
-    <visual name="sonar1_visual">
-      <origin xyz="0 0 0" rpy="0 0 -1.570796327"/>
-      <geometry>
-        <mesh filename="package://jet_description/meshes/Sonar_1.dae"/>
-      </geometry>
-    </visual>
-    <inertial>
-      <mass value="1e-5" />
-      <origin xyz="0 0 0" rpy="0 0 -1.570796327"/>
-      <inertia ixx="1e-6" ixy="0" ixz="0" iyy="1e-6" iyz="0" izz="1e-6" />
-    </inertial>
-  </link>
-  <!-- Sonar_Sensor_2 -->
-  <link name="sonar2_link">
-    <collision name="collision">
-      <origin xyz="0 0 0" rpy="0 0 -1.570796327"/>
-      <geometry>
-        <mesh filename="package://jet_description/meshes/Sonar_2.dae"/>
-      </geometry>
-    </collision>
-    <visual name="sonar2_visual">
-      <origin xyz="0 0 0" rpy="0 0 -1.570796327"/>
-      <geometry>
-        <mesh filename="package://jet_description/meshes/Sonar_2.dae"/>
-      </geometry>
-    </visual>
-    <inertial>
-      <mass value="1e-5" />
-      <origin xyz="0 0 0" rpy="0 0 -1.570796327"/>
-      <inertia ixx="1e-6" ixy="0" ixz="0" iyy="1e-6" iyz="0" izz="1e-6" />
-    </inertial>
-  </link>
-  <!-- Sonar_Sensor_3 -->
-  <link name="sonar3_link">
-    <collision name="collision">
-      <origin xyz="0 0 0" rpy="0 0 -1.570796327"/>
-      <geometry>
-        <mesh filename="package://jet_description/meshes/Sonar_3.dae"/>
-      </geometry>
-    </collision>
-    <visual name="sonar2_visual">
-      <origin xyz="0 0 0" rpy="0 0 -1.570796327"/>
-      <geometry>
-        <mesh filename="package://jet_description/meshes/Sonar_3.dae"/>
-      </geometry>
-    </visual>
-    <inertial>
-      <mass value="1e-5" />
-      <origin xyz="0 0 0" rpy="0 0 -1.570796327"/>
-      <inertia ixx="1e-6" ixy="0" ixz="0" iyy="1e-6" iyz="0" izz="1e-6" />
-    </inertial>
-  </link>
-  <!-- Liadar -->
-  <link name="hokuyo">
-    <collision name="collision">
-      <origin xyz="-0.0225 0 -0.02" rpy="0 0 3.141592654"/>
-      <geometry>
-        <mesh filename="package://jet_description/meshes/Hokuyo.dae"/>
-      </geometry>
-    </collision>
-    <visual name="hokuyo_visual">
-      <origin xyz="-0.0225 0 -0.02" rpy="0 0 3.141592654"/>
-      <geometry>
-        <mesh filename="package://jet_description/meshes/Hokuyo.dae"/>
-      </geometry>
-    </visual>
-    <inertial>
-      <mass value="1e-5" />
-      <origin xyz="-0.0225 0 -0.02" rpy="0 0 3.141592654"/>
-      <inertia ixx="1e-6" ixy="0" ixz="0" iyy="1e-6" iyz="0" izz="1e-6" />
-    </inertial>
-  </link>
-  <!-- IMU -->
-  <link name="IMU_link">
-    <collision name="collision">
-      <origin xyz="0 0 0" rpy="0 0 0"/>
-      <geometry>
-        <mesh filename="package://jet_description/meshes/IMU.dae"/>
-      </geometry>
-    </collision>
-    <visual name="IMU_visual">
-      <origin xyz="0 0 0" rpy="0 0 0"/>
-      <geometry>
-        <mesh filename="package://jet_description/meshes/IMU.dae"/>
-      </geometry>
-    </visual>
-    <inertial>
-      <mass value="1e-6"/>
-      <origin rpy="0 0 0" xyz="0 0 0"/>
-      <inertia ixx="0" ixy="0" ixz="0" iyy="0" iyz="0" izz="0"/>
-    </inertial>
-  </link>
-<!--........................JOINTS........................-->
-  <!-- Left Wheel Joint -->
-  <joint type="continuous" name="left_wheel_joint">
-    <origin xyz="0.15 -0.075 0.02" rpy="0 0 0"/>
-    <child link="left_wheel"/>
-    <parent link="chassis"/>
-    <axis xyz="1 0 0" rpy="0 0 0"/>
-    <limit effort="100" velocity="100"/>
-    <joint_properties damping="3.0" friction="0.0"/>
-  </joint>
-  <!-- Right Wheel Joint -->
-  <joint type="continuous" name="right_wheel_joint">
-    <origin xyz="-0.15 -0.075 0.02" rpy="0 0 0"/>
-    <child link="right_wheel"/>
-    <parent link="chassis"/>
-    <axis xyz="1 0 0" rpy="0 0 0"/>
-    <limit effort="100" velocity="100"/>
-    <joint_properties damping="3.0" friction="0.0"/>
-  </joint>
-  <!-- Caster Link Joint -->
-  <joint type="continuous" name="caster_joint">
-    <origin xyz="0 0.1 0.005" rpy="0 0 0"/>
-    <child link="caster_link"/>
-    <parent link="chassis"/>
-    <axis xyz="0 0 1" rpy="0 0 0"/>
-    <limit effort="100" velocity="100"/>
-    <joint_properties damping="0.0" friction="0.0"/>
-  </joint>
-  <!-- Caster Wheel Joint -->
   <joint type="continuous" name="caster_turn">
     <origin xyz="0 0.02 -0.0375" rpy="0 0 0"/>
@@ -276,8 +148,19 @@
     <parent link="caster_link"/>
     <axis xyz="1 0 0" rpy="0 0 0"/>
-    <limit effort="100" velocity="100"/>
-    <joint_properties damping="0.0" friction="0.0"/>
-  </joint>
-  <!-- Camera_Joint -->
+  </joint>
+  <!--................................Camera..................................-->
+  <link name="camera">
+    <visual name="camera_visual">
+      <origin xyz="0 0 0" rpy="0 1.570796327 0"/>
+      <geometry>
+        <mesh filename="package://jet_description/meshes/Camera.dae"/>
+      </geometry>
+    </visual>
+    <inertial>
+      <origin xyz="0 0 0" rpy="0 0 0"/>
+      <mass value="0.1" />
+      <inertia ixx="0" ixy="0" ixz="0" iyy="0" iyz="0" izz="0" />
+    </inertial>
+  </link>
   <joint name="camera_joint" type="fixed">
     <axis xyz="0 0 0" rpy="0 0 0" />
@@ -286,5 +169,58 @@
     <child link="camera"/>
   </joint>
-  <!-- Sonar_1_Joint -->
+  <!--............................Liadar................................-->
+  <link name="hokuyo">
+    <visual name="hokuyo_visual">
+      <origin xyz="0 0 -0.015" rpy="0 0 0"/>
+      <geometry>
+        <mesh filename="package://jet_description/meshes/Hokuyo.dae"/>
+      </geometry>
+    </visual>
+    <inertial>
+      <mass value="0.25" />
+      <origin xyz="0 0 0" rpy="0 0 0"/>
+      <inertia ixx="0" ixy="0" ixz="0" iyy="0" iyz="0" izz="0" />
+    </inertial>
+  </link>
+  <joint name="hokuyo_joint" type="fixed">
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